Commit message: Config and launch file fixes

File: config/aria_panda_arm.xacro (robot description, xacro)
@@ -18,21 +18,22 @@
       </visual>
       <collision>
-        <origin xyz="-0.075 0 0.06" rpy="0 ${pi/2} 0"/>
-        <geometry>
-          <cylinder radius="${0.06+safety_distance}" length="0.03" />
-        </geometry>
-      </collision>
-      <collision>
+        <origin xyz="-0.075 0 0.07" rpy="0 0 0"/>
+        <geometry>
+          <!--cylinder radius="${0.006+safety_distance}" length="0.03" /-->
+          <box size=".16 .16 .14"/>
+        </geometry>
+      </collision>
+      <!--collision>
         <origin xyz="-0.06 0 0.06" rpy="0 0 0"/>
         <geometry>
-          <sphere radius="${0.06+safety_distance}" />
-        </geometry>
-      </collision>
-      <collision>
+          <sphere radius="${0.006+safety_distance}" />
+        </geometry>
+      </collision-->
+      <!--collision>
         <origin xyz="-0.09 0 0.06" rpy="0 0 0"/>
         <geometry>
           <sphere radius="${0.06+safety_distance}" />
         </geometry>
-      </collision>
+      </collision-->
     </link>
     <link name="${arm_id}_link1">
@@ -48,10 +49,10 @@
         </geometry>
       </collision>
-      <collision>
+      <!--collision>
         <origin xyz="0 0 -0.333" rpy="0 0 0"/>
         <geometry>
           <sphere radius="${0.06+safety_distance}" />
         </geometry>
-      </collision>
+      </collision-->
       <collision>
         <origin xyz="0 0 -0.05" rpy="0 0 0"/>

File: config/panda_arm.urdf.xacro (robot description, xacro)
@@ -7,9 +7,9 @@
   <xacro:unless value="$(arg gazebo)">
     <!-- Create a URDF for a real hardware -->
-    <xacro:include filename="$(find vicon_franka_integration)/robots/aria_panda_arm.xacro" />
-    <xacro:panda_arm arm_id="${arm_id}" safety_distance="0.02"/>
+    <xacro:include filename="$(find manipulation_interface)/config/aria_panda_arm.xacro" />
+    <xacro:panda_arm arm_id="$(arg arm_id)" safety_distance="0.02"/>
     <xacro:if value="$(arg hand)">
-      <xacro:include filename="$(find vicon_franka_integration)/robots/aria_franka_hand.xacro"/>
-      <xacro:hand ns="${arm_id}" rpy="0 0 ${-pi/4}" connected_to="${arm_id}_link8" safety_distance="0.02"/>
+      <xacro:include filename="$(find manipulation_interface)/config/aria_franka_hand.xacro"/>
+      <xacro:hand ns="$(arg arm_id)" rpy="0 0 ${-pi/4}" connected_to="$(arg arm_id)_link8" safety_distance="0.02"/>
     </xacro:if>
   </xacro:unless>
@@ -20,9 +20,9 @@
     <xacro:include filename="$(find franka_description)/robots/utils.xacro" />
     <xacro:include filename="$(find franka_description)/robots/panda_gazebo.xacro" />
-    <xacro:panda_arm arm_id="${arm_id}" />
+    <xacro:panda_arm arm_id="$(arg arm_id)" />
     <xacro:if value="$(arg hand)">
-      <xacro:hand ns="${arm_id}" rpy="0 0 ${-pi/4}" connected_to="${arm_id}_link8" />
-      <xacro:gazebo-joint joint="${arm_id}_finger_joint1" transmission="hardware_interface/EffortJointInterface" />
-      <xacro:gazebo-joint joint="${arm_id}_finger_joint2" transmission="hardware_interface/EffortJointInterface" />
+      <xacro:hand ns="$(arg arm_id)" rpy="0 0 ${-pi/4}" connected_to="$(arg arm_id)_link8" />
+      <xacro:gazebo-joint joint="$(arg arm_id)_finger_joint1" transmission="hardware_interface/EffortJointInterface" />
+      <xacro:gazebo-joint joint="$(arg arm_id)_finger_joint2" transmission="hardware_interface/EffortJointInterface" />
     </xacro:if>
     <!-- Gazebo requires a joint to a link called "world" for statically mounted robots -->
@@ -31,21 +31,21 @@
       <origin xyz="$(arg xyz)" rpy="$(arg rpy)" />
       <parent link="world" />
-      <child  link="${arm_id}_link0" />
+      <child  link="$(arg arm_id)_link0" />
     </joint>
-    <xacro:gazebo-joint joint="${arm_id}_joint1" transmission="hardware_interface/EffortJointInterface" />
-    <xacro:gazebo-joint joint="${arm_id}_joint2" transmission="hardware_interface/EffortJointInterface" />
-    <xacro:gazebo-joint joint="${arm_id}_joint3" transmission="hardware_interface/EffortJointInterface" />
-    <xacro:gazebo-joint joint="${arm_id}_joint4" transmission="hardware_interface/EffortJointInterface" />
-    <xacro:gazebo-joint joint="${arm_id}_joint5" transmission="hardware_interface/EffortJointInterface" />
-    <xacro:gazebo-joint joint="${arm_id}_joint6" transmission="hardware_interface/EffortJointInterface" />
-    <xacro:gazebo-joint joint="${arm_id}_joint7" transmission="hardware_interface/EffortJointInterface" />
-    <xacro:transmission-franka-state arm_id="${arm_id}" />
-    <xacro:transmission-franka-model arm_id="${arm_id}"
-       root="${arm_id}_joint1"
-       tip="${arm_id}_joint8"
+    <xacro:gazebo-joint joint="$(arg arm_id)_joint1" transmission="hardware_interface/EffortJointInterface" />
+    <xacro:gazebo-joint joint="$(arg arm_id)_joint2" transmission="hardware_interface/EffortJointInterface" />
+    <xacro:gazebo-joint joint="$(arg arm_id)_joint3" transmission="hardware_interface/EffortJointInterface" />
+    <xacro:gazebo-joint joint="$(arg arm_id)_joint4" transmission="hardware_interface/EffortJointInterface" />
+    <xacro:gazebo-joint joint="$(arg arm_id)_joint5" transmission="hardware_interface/EffortJointInterface" />
+    <xacro:gazebo-joint joint="$(arg arm_id)_joint6" transmission="hardware_interface/EffortJointInterface" />
+    <xacro:gazebo-joint joint="$(arg arm_id)_joint7" transmission="hardware_interface/EffortJointInterface" />
+    <xacro:transmission-franka-state arm_id="$(arg arm_id)" />
+    <xacro:transmission-franka-model arm_id="$(arg arm_id)"
+       root="$(arg arm_id)_joint1"
+       tip="$(arg arm_id)_joint8"
      />
     <gazebo>
       <plugin name="gazebo_ros_control" filename="libgazebo_ros_control.so">
-        <robotNamespace>${arm_id}</robotNamespace>
+        <robotNamespace>$(arg arm_id)</robotNamespace>
         <controlPeriod>0.001</controlPeriod>
         <robotSimType>franka_gazebo/FrankaHWSim</robotSimType>
