Commit message: Panda xacro launch and manipulator node overhaul WIP

File: config/franka_hand.xacro (robot description, xacro)
@@ -19,5 +19,5 @@
         <origin xyz="0 0 0.02" rpy="0 ${pi/2} ${pi/2}"/>
         <geometry>
-          <cylinder radius="${0.02+safety_distance}" length="0.2" />
+          <cylinder radius="${0.026+safety_distance}" length="0.2" />
         </geometry>
       </collision>
@@ -25,5 +25,5 @@
         <origin xyz="0 -0.1 0.02" rpy="0 0 0"/>
         <geometry>
-          <sphere radius="${0.02+safety_distance}"  />
+          <sphere radius="${0.026+safety_distance}"  />
         </geometry>
       </collision>
@@ -31,5 +31,5 @@
         <origin xyz="0 0.1 0.02" rpy="0 0 0"/>
         <geometry>
-          <sphere radius="${0.02+safety_distance}"  />
+          <sphere radius="${0.026+safety_distance}"  />
         </geometry>
       </collision>

File: config/panda_arm.urdf.xacro (robot description, xacro)
@@ -10,5 +10,5 @@
     <xacro:panda_arm arm_id="$(arg arm_id)" safety_distance="0.02"/>
     <xacro:if value="$(arg hand)">
-      <xacro:include filename="$(find manipulation_interface)/config/aria_franka_hand.xacro"/>
+      <xacro:include filename="$(find manipulation_interface)/config/franka_hand.xacro"/>
       <xacro:hand ns="$(arg arm_id)" rpy="0 0 ${-pi/4}" connected_to="$(arg arm_id)_link8" safety_distance="0.02"/>
     </xacro:if>

Commit message: Minor edits to help experiments

File: config/franka_hand.xacro (robot description, xacro)
@@ -44,5 +44,5 @@
         <geometry>
           <!--sphere radius="${0.02+safety_distance}"  /-->
-	  <box size=".03 .04 .07"/>
+	  <box size=".02 .02 .06"/>
         </geometry>
       </collision>
@@ -51,5 +51,5 @@
         <geometry>
           <!--sphere radius="${0.02+safety_distance}"  /-->
-	  <box size=".03 .04 .07"/>
+	  <box size=".02 .02 .06"/>
         </geometry>
       </collision>
