Commit message: Fix config files

File: config/dont_need_custom_panda_arm.xacro (robot description, xacro)
@@ -18,22 +18,22 @@
       </visual>
       <collision>
-        <origin xyz="-0.075 0 0.07" rpy="0 0 0"/>
-        <geometry>
-          <!--cylinder radius="${0.006+safety_distance}" length="0.03" /-->
-          <box size=".16 .16 .14"/>
-        </geometry>
-      </collision>
-      <!--collision>
+        <origin xyz="-0.075 0 0.06" rpy="0 ${pi/2} 0"/>
+        <geometry>
+          <!-- <cylinder radius="${0.06+safety_distance}" length="0.03" /> -->
+          <box size="0.16 .16 .14"/>
+        </geometry>
+      </collision>
+      <!-- <collision>
         <origin xyz="-0.06 0 0.06" rpy="0 0 0"/>
         <geometry>
-          <sphere radius="${0.006+safety_distance}" />
-        </geometry>
-      </collision-->
-      <!--collision>
+          <sphere radius="${0.06+safety_distance}" />
+        </geometry>
+      </collision>
+      <collision>
         <origin xyz="-0.09 0 0.06" rpy="0 0 0"/>
         <geometry>
           <sphere radius="${0.06+safety_distance}" />
         </geometry>
-      </collision-->
+      </collision> -->
     </link>
     <link name="${arm_id}_link1">
@@ -49,10 +49,10 @@
         </geometry>
       </collision>
-      <!--collision>
+      <!-- <collision>
         <origin xyz="0 0 -0.333" rpy="0 0 0"/>
         <geometry>
           <sphere radius="${0.06+safety_distance}" />
         </geometry>
-      </collision-->
+      </collision> -->
       <collision>
         <origin xyz="0 0 -0.05" rpy="0 0 0"/>
@@ -63,4 +63,5 @@
     </link>
     <joint name="${arm_id}_joint1" type="revolute">
+      <!-- <safety_controller k_position="100.0" k_velocity="40.0" soft_lower_limit="-2.8973" soft_upper_limit="2.8973"/> -->
 	    <safety_controller k_position="100.0" k_velocity="40.0" soft_lower_limit="${-2.8973 + soft_limit_offset}" soft_upper_limit="${2.8973 - soft_limit_offset}"/>
       <origin rpy="0 0 0" xyz="0 0 0.333"/>
@@ -279,5 +280,5 @@
     </link>
     <joint name="${arm_id}_joint7" type="revolute">
-	    <safety_controller k_position="100.0" k_velocity="40.0" soft_lower_limit="${-2.8973 + soft_limit_offset}" soft_upper_limit="${2.8973 - soft_limit_offset}"/>
+      <safety_controller k_position="100.0" k_velocity="40.0" soft_lower_limit="-2.8973" soft_upper_limit="2.8973"/>
       <origin rpy="${pi/2} 0 0" xyz="0.088 0 0"/>
       <parent link="${arm_id}_link6"/>

File: config/panda_arm.urdf.xacro (robot description, xacro)
@@ -7,8 +7,8 @@
   <xacro:unless value="$(arg gazebo)">
     <!-- Create a URDF for a real hardware -->
-    <xacro:include filename="$(find manipulation_interface)/config/aria_panda_arm.xacro" />
+    <xacro:include filename="$(find manipulation_interface)/config/custom_panda_arm.xacro" />
     <xacro:panda_arm arm_id="$(arg arm_id)" safety_distance="0.02"/>
     <xacro:if value="$(arg hand)">
-      <xacro:include filename="$(find manipulation_interface)/config/franka_hand.xacro"/>
+      <xacro:include filename="$(find manipulation_interface)/config/custom_hand.xacro"/>
       <xacro:hand ns="$(arg arm_id)" rpy="0 0 ${-pi/4}" connected_to="$(arg arm_id)_link8" safety_distance="0.02"/>
     </xacro:if>
